Commit message: 修改steady_tray_env_cfg.py为残差输出

File: source/steadytray/steadytray/assets/g1_29dof.urdf (robot description, URDF)
Before this commit: robot g1_29dof, 37 links, 36 joints
Links:
- link left_rubber_hand: geometry collision box size=0.08 0.03 0.08; visual mesh filename=meshes/left_rubber_hand.STL
- link right_rubber_hand: geometry collision box size=0.08 0.03 0.08; visual mesh filename=meshes/right_rubber_hand.STL
